File: BOOST/BOOST.kicad_sch (KiCad schematic)
At the start: 268 parts, among them M1 HYG180N10, M10 HYG180N10, M2 HYG180N10, M3 HYG180N10, M4 HYG180N10, M5 HYG180N10, M6 HYG180N10, M7 HYG180N10, M8 HYG180N10, M9 HYG180N10, Q1 PNP, U1 L78L05_SOT89, U10 UCC21520DW, U101 74HC00, U102 74HC00, U103 74HC00, U104 74HC14, U105 74HC14, U106 CD74HC4066, U11 MCP6241, U12 MCP6241, U13 MCP6241, U14 MCP6561, U15 UCC21520DW, U16 LM2940_12, U17 L78L05_SOT89, U18 4017, U19 UCC21520DW, U2 MCP6561, U20 74HC14, U21 MCP6561, U22 MCP6241, U23 MCP6241, U24 MCP6241, U25 INA241A3xD, U26 MCP4451-xxxx-ST, U27 74HC00, U28 74HC4051, U3 MCP6241, U4 MCP6561, U5 MCP6561, U6 MCP6241, U7 MCP6241, U8 UCC21520DW, U9 MCP6561-OT

Commit message: added connector and fixed more footprints
Parts:
- removed D16: 100W_LED_RED, symbol ltspice:diode
- removed D17: 100W_LED_BLUE, symbol ltspice:diode
- removed D18: 100W_LED_GREEN, symbol ltspice:diode
- removed U20: 74HC14, symbol 74xx:74HC14
- removed U27: 74HC00, symbol 74xx:74HC00
- removed U9: MCP6561-OT, Package_TO_SOT_SMD:SOT-23-5, symbol Comparator:MCP6561-OT
- added C104: 100n, Capacitor_SMD:C_0603_1608Metric, symbol ltspice:cap
- added J1, J2: Conn_01x01_Pin, MountingHole:MountingHole_4.3mm_M4_Pad_TopBottom, symbol Connector:Conn_01x01_Pin
- added J3, J4, J5, J6, J7, J8: Conn_01x01_Pin, TestPoint:TestPoint_THTPad_4.0x4.0mm_Drill2.0mm, symbol Connector:Conn_01x01_Pin
- added J9: Conn_01x10, Connector_PinHeader_2.54mm:PinHeader_1x10_P2.54mm_Vertical, symbol Connector_Generic:Conn_01x10
- added unit 5 of U26
- added unit 4 of U26
- L1: footprint (none) -> CSCF3218-6R8MC:IND_CSCF3218-6R8MC
- M1, M10, M2, M3, M4, M5, M6, M7, M8, M9: footprint (none) -> Package_TO_SOT_THT:TO-220-3_Horizontal_TabDown
- U18, U28: footprint (none) -> Package_SO:SOIC-16_3.9x9.9mm_P1.27mm
Connections:
- net 5V: now also C104.1, J9.9 (Pin_9), U26.17 (VDD)
- net GND: now also C104.2, J2.1 (Pin_1), J9.10 (Pin_10), U26.15 (~{RESET}), U26.7 (VSS)
- net IREF1: now also J9.4 (Pin_4)
- net IREF2: now also J9.5 (Pin_5)
- net IREF3: now also J9.6 (Pin_6)
- net Output1_drain: now also J4.1 (Pin_1)
- net Output2_drain: now also J7.1 (Pin_1)
- net Output3_drain: now also J6.1 (Pin_1)
- net Vin: now also J1.1 (Pin_1)
- net Vout_1: now also J3.1 (Pin_1)
- net Vout_2: now also J8.1 (Pin_1)
- net Vout_3: now also J5.1 (Pin_1)
- net Vref_1_arduino: now also J9.1 (Pin_1)
- net Vref_2_arduino: now also J9.2 (Pin_2)
- net Vref_3_arduino: now also J9.3 (Pin_3)
- new net SCL: J9.7 (Pin_7), U26.5 (SCL)
- new net SDA: J9.8 (Pin_8), U26.6 (SDA)
- no-connect marks 0 -> 10
