File: BOOST/BOOST.kicad_sch (KiCad schematic)
At the start: 272 parts, among them J1 Conn_01x01_Pin, J2 Conn_01x01_Pin, J3 Conn_01x01_Pin, J4 Conn_01x01_Pin, J5 Conn_01x01_Pin, J6 Conn_01x01_Pin, J7 Conn_01x01_Pin, J8 Conn_01x01_Pin, J9 Conn_01x10, M1 HYG180N10, M10 HYG180N10, M2 HYG180N10, M3 HYG180N10, M4 HYG180N10, M5 HYG180N10, M6 HYG180N10, M7 HYG180N10, M8 HYG180N10, M9 HYG180N10, Q1 PNP, U1 L78L05_SOT89, U10 UCC21520DW, U101 74HC00, U102 74HC00, U103 74HC00, U104 74HC14, U105 74HC14, U106 CD74HC4066, U11 MCP6241, U12 MCP6241, U13 MCP6241, U14 MCP6561, U15 UCC21520DW, U16 LM2940_12, U17 L78L05_SOT89, U18 4017, U19 UCC21520DW, U2 MCP6561, U21 MCP6561, U22 MCP6241, U23 MCP6241, U24 MCP6241, U25 INA241A3xD, U26 MCP4451-xxxx-ST, U28 74HC4051, U3 MCP6241, U4 MCP6561, U5 MCP6561, U6 MCP6241, U7 MCP6241, U8 UCC21520DW

Commit message: onto pcb editor
Parts:
- removed C41, C44, C45: 1n, Capacitor_SMD:C_0603_1608Metric, symbol ltspice:cap
- added R102, R103, R104, R99: 10k, Resistor_SMD:R_0603_1608Metric, symbol ltspice:res
- added unit 3 of U103
- added unit 4 of U103
- added unit 4 of U105
- added unit 6 of U105
- added unit 5 of U105
- added unit 3 of U105
- added unit 4 of U106
Connections:
- net 5V: now also R103.1
- net GATE_M1: now also R104.1
- net GATE_M4: now also R73.2
- net GATE_M5: now also R74.2
- net GND: now also R102.2, R104.2, R99.2; no longer U26.15 (~{RESET})
- net at D22.1 (-), R59.2, U8.10 (OUTB): no longer R74.2
- net at D13.1 (-), R47.2, U8.15 (OUTA): no longer R73.2
- net at U26.16 (A1): now also R99.1
- net at U26.4 (HVC/A0): now also R102.1
- new net: R103.2, U26.15 (~{RESET})
- no-connect marks 10 -> 27
Other:
- moved on the sheet: R73, R74
